Commit message: Changed URDF

File: description/urdf/mercury_description.urdf.xacro (robot description, xacro)
@@ -12,5 +12,5 @@
   <xacro:create_link
       link_name="link_1"
-      xyz_offset="0 0 0.1255"
+      xyz_offset="0 0 0"
       rpy_offset="0 0 0"
       mesh_name="ROS2_J1"
@@ -18,5 +18,5 @@
   <xacro:create_link
       link_name="link_2"
-      xyz_offset="0 0.168 0"
+      xyz_offset="0 0 0"
       rpy_offset="0 0 0"
       mesh_name="ROS2_J2"
@@ -24,5 +24,5 @@
   <xacro:create_link
       link_name="link_3"
-      xyz_offset="0 0.020 0"
+      xyz_offset="0 0 0"
       rpy_offset="0 0 0"
       mesh_name="ROS2_J3"
@@ -30,5 +30,5 @@
   <xacro:create_link
       link_name="link_4"
-      xyz_offset="0 0.153 0"
+      xyz_offset="0 0 0"
       rpy_offset="0 0 0"
       mesh_name="ROS2_J4"
@@ -36,5 +36,5 @@
   <xacro:create_link
       link_name="link_5"
-      xyz_offset="0 0 0.133"
+      xyz_offset="0 0 0"
       rpy_offset="0 0 0"
       mesh_name="ROS2_J5"
@@ -42,5 +42,5 @@
   <xacro:create_link
       link_name="link_6"
-      xyz_offset="0 0.1005 0"
+      xyz_offset="0 0 0"
       rpy_offset="0 0 0"
       mesh_name="ROS2_J6"
@@ -66,5 +66,5 @@
     <parent link="link_1"/>
     <child link="link_2"/>
-    <origin xyz="0 0 0.1255" rpy="0 0 0"/>
+    <origin xyz="0 0 0" rpy="0 ${-pi/2} 0"/>
     <axis xyz="0 1 0"/>
     <limit effort="1000.0" lower="${-pi}" upper="${pi}" velocity="2.5"/>
@@ -73,5 +73,5 @@
     <parent link="link_2"/>
     <child link="link_3"/>
-    <origin xyz="0 0 0.320" rpy="0 ${pi} ${pi+pi/2}"/>
+    <origin xyz="0 0 0" rpy="0 0 0"/>
     <axis xyz="0 1 0"/>
     <limit effort="1000.0" lower="${-pi}" upper="${pi}" velocity="2.5"/>
@@ -80,5 +80,5 @@
     <parent link="link_3"/>
     <child link="link_4"/>
-    <origin xyz="0 0 0.315" rpy="0 ${pi} ${pi+pi/6}"/>
+    <origin xyz="0 0 0" rpy="0 0 0"/>
     <axis xyz="0 1 0"/>
     <limit effort="1000.0" lower="${-pi}" upper="${pi}" velocity="2.5"/>
@@ -87,5 +87,5 @@
     <parent link="link_4"/>
     <child link="link_5"/>
-    <origin xyz="0 0 0.133" rpy="${pi/2} ${pi} ${pi/2}"/>
+    <origin xyz="0 0 0" rpy="0 0 0"/>
     <axis xyz="0 0 1"/>
     <limit effort="1000.0" lower="${-pi}" upper="${pi}" velocity="2.5"/>
@@ -94,5 +94,5 @@
     <parent link="link_5"/>
     <child link="link_6"/>
-    <origin xyz="0 0 0.133" rpy="0 ${-pi/2} 0"/>
+    <origin xyz="0 0 0" rpy="0 0 0"/>
     <axis xyz="0 1 0"/>
     <limit effort="1000.0" lower="${-pi}" upper="${pi}" velocity="2.5"/>

Commit message: Correctet Origins

File: description/urdf/mercury_description.urdf.xacro (robot description, xacro)
@@ -59,5 +59,5 @@
     <parent link="base_link"/>
     <child link="link_1"/>
-    <origin xyz="0 0 0" rpy="0 0 0"/>
+    <origin xyz="0 0 0.117" rpy="0 0 0"/>
     <axis xyz="0 0 1"/>
     <limit effort="1000.0" lower="${-pi}" upper="${pi}" velocity="2.5"/>
@@ -66,6 +66,6 @@
     <parent link="link_1"/>
     <child link="link_2"/>
-    <origin xyz="0 0 0" rpy="0 ${-pi/2} 0"/>
-    <axis xyz="0 1 0"/>
+    <origin xyz="-0.081 0 0.101" rpy="0 ${-pi/2} 0"/>
+    <axis xyz="0 0 1"/>
     <limit effort="1000.0" lower="${-pi}" upper="${pi}" velocity="2.5"/>
   </joint>
@@ -73,6 +73,6 @@
     <parent link="link_2"/>
     <child link="link_3"/>
-    <origin xyz="0 0 0" rpy="0 0 0"/>
-    <axis xyz="0 1 0"/>
+    <origin xyz="0.35 0 -0.0035" rpy="${pi} 0 0"/>
+    <axis xyz="0 0 1"/>
     <limit effort="1000.0" lower="${-pi}" upper="${pi}" velocity="2.5"/>
   </joint>
@@ -80,6 +80,6 @@
     <parent link="link_3"/>
     <child link="link_4"/>
-    <origin xyz="0 0 0" rpy="0 0 0"/>
-    <axis xyz="0 1 0"/>
+    <origin xyz="0.0805 0 0.0775" rpy="${pi} ${pi/2} 0"/>
+    <axis xyz="0 0 1"/>
     <limit effort="1000.0" lower="${-pi}" upper="${pi}" velocity="2.5"/>
   </joint>
@@ -87,5 +87,5 @@
     <parent link="link_4"/>
     <child link="link_5"/>
-    <origin xyz="0 0 0" rpy="0 0 0"/>
+    <origin xyz="0 0 0.2695" rpy="0 ${-pi/2} 0"/>
     <axis xyz="0 0 1"/>
     <limit effort="1000.0" lower="${-pi}" upper="${pi}" velocity="2.5"/>
@@ -94,6 +94,6 @@
     <parent link="link_5"/>
     <child link="link_6"/>
-    <origin xyz="0 0 0" rpy="0 0 0"/>
-    <axis xyz="0 1 0"/>
+    <origin xyz="0.1705 0 0" rpy="0 ${pi/2} 0"/>
+    <axis xyz="0 0 1"/>
     <limit effort="1000.0" lower="${-pi}" upper="${pi}" velocity="2.5"/>
   </joint>
