Commit message: Fixes

File: description/urdf/inc/create_link.xacro (robot description, xacro)
@@ -10,5 +10,5 @@
         <origin xyz="${xyz_offset}" rpy="${rpy_offset}"/>
         <geometry>
-          <mesh filename="package://tr_robot/meshes/${mesh_name}.stl" scale="0.001 0.001 0.001"/>
+          <mesh filename="package://tr_robot/description/meshes/${mesh_name}.stl" scale="0.001 0.001 0.001"/>
         </geometry>
       </visual>
@@ -16,5 +16,5 @@
         <origin xyz="${xyz_offset}" rpy="${rpy_offset}"/>
         <geometry>
-          <mesh filename="package://tr_robot/meshes/${mesh_name}.stl" scale="0.001 0.001 0.001"/>
+          <mesh filename="package://tr_robot/description/meshes/${mesh_name}.stl" scale="0.001 0.001 0.001"/>
         </geometry>
       </collision>

File: description/urdf/mercury.urdf.xacro (robot description, xacro)
@@ -5,7 +5,7 @@
   <!-- create link fixed to the "world" -->
   <link name="world"/>
-  <xacro:r6bot_description/>
+  <xacro:mercury_description/>
   <!-- Import mercury ros2_control description -->
-  <xacro:include filename="$(find description)/ros2_control/mercury.ros2_control.xacro" />
-  <xacro:mercury_ros2_control name="mercury"/>
+  <!-- <xacro:include filename="$(find description)/ros2_control/mercury.ros2_control.xacro" />
+  <xacro:mercury_ros2_control name="mercury"/> -->
 </robot>

File: description/urdf/mercury_description.urdf.xacro (robot description, xacro)
@@ -8,5 +8,5 @@
       xyz_offset="0 0 0"
       rpy_offset="0 0 0"
-      mesh_name="ROS2_J0"
+      mesh_name="ROS2_Base"
   />
   <xacro:create_link
@@ -80,5 +80,5 @@
     <parent link="link_3"/>
     <child link="link_4"/>
-    <origin xyz="0.0805 0 0.0775" rpy="${pi} ${pi/2} 0"/>
+    <origin xyz="0.0805 0 0.0775" rpy="0 ${pi/2} 0"/>
     <axis xyz="0 0 1"/>
     <limit effort="1000.0" lower="${-pi}" upper="${pi}" velocity="2.5"/>
